File: usb_c.kicad_sch (KiCad schematic)
At the start: 23 parts, among them J1 USB_C_Receptacle, U1 MIC5363-3.3YMT, U2 HD3SS3220, U3 MG2040

Commit message: Changes:
-fix led order
-fix transistor routing
-modify usb hub strapping and fix crystal footprint
-remove copper under sd pads
-routing cleanup
-change revision to 1.1

Signed-off-by: Dominik Sliwa <dominik@sliwa.io>
Other:
- company: (none) -> SliwaIO
- title: (none) -> SDReWire
Changed lines of the file:
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@@
-(kicad_sch (version 20201015) (generator eeschema)
-  (page 1 5)
+(kicad_sch (version 20210126) (generator eeschema)
   (paper "A4")
+  (title_block
+    (title "SDReWire")
+    (rev "1.1")
+    (company "SliwaIO")
+  )
   (junction (at 29.972 151.13) (diameter 1.016) (color 0 0 0 0))
   (junction (at 51.562 97.282) (diameter 1.016) (color 0 0 0 0))
@@
   (junction (at 148.59 47.752) (diameter 1.016) (color 0 0 0 0))
   (junction (at 152.4 38.862) (diameter 1.016) (color 0 0 0 0))
+  (no_connect (at 49.022 139.192))
   (no_connect (at 49.022 141.732))
   (no_connect (at 55.372 31.242))
+  (no_connect (at 55.372 36.322))
+  (no_connect (at 55.372 41.402))
+  (no_connect (at 55.372 46.482))
   (no_connect (at 55.372 51.562))
+  (no_connect (at 135.382 126.492))
+  (no_connect (at 135.382 129.032))
+  (no_connect (at 135.382 141.732))
   (no_connect (at 135.382 144.272))
-  (no_connect (at 55.372 46.482))
+  (no_connect (at 135.382 146.812))
   (no_connect (at 135.382 151.892))
-  (no_connect (at 55.372 41.402))
-  (no_connect (at 135.382 129.032))
-  (no_connect (at 55.372 36.322))
-  (no_connect (at 135.382 141.732))
-  (no_connect (at 135.382 126.492))
-  (no_connect (at 135.382 146.812))
-  (no_connect (at 49.022 139.192))
   (no_connect (at 135.382 154.432))
   (wire (pts (xy 26.162 151.13) (xy 26.162 149.352))
@@
       (effects (font (size 1.27 1.27)) hide)
     )
+    (pin "1")
   )
   (symbol (lib_id "power:+5V") (at 99.822 36.83 0) (unit 1)
@@
       (effects (font (size 1.27 1.27)) hide)
     )
+    (pin "1")
   )
   (symbol (lib_id "power:+5V") (at 107.442 97.282 0) (unit 1)
@@
       (effects (font (size 1.27 1.27)) hide)
     )
+    (pin "1")
   )
   (symbol (lib_id "power:+3V3") (at 112.522 97.282 0) (unit 1)
@@
       (effects (font (size 1.27 1.27)) hide)
     )
+    (pin "1")
   )
   (symbol (lib_id "power:+5V") (at 149.352 134.112 270) (unit 1)
@@
       (effects (font (size 1.27 1.27)) hide)
     )
+    (pin "1")
   )
   (symbol (lib_id "power:+3V3") (at 149.352 139.192 270) (unit 1)
@@
       (effects (font (size 1.27 1.27)) hide)
     )
+    (pin "1")
   )
   (symbol (lib_id "power:+3V3") (at 157.48 36.322 0) (unit 1)
@@
       (effects (font (size 1.27 1.27)) hide)
     )
+    (pin "1")
   )
   (symbol (lib_id "power:+3V3") (at 203.2 30.48 0) (unit 1)
@@
       (effects (font (size 1.27 1.27)) hide)
     )
+    (pin "1")
   )
   (symbol (lib_id "power:GND") (at 29.972 153.162 0) (unit 1)
@@
       (effects (font (size 1.27 1.27)) hide)
     )
+    (pin "1")
   )
   (symbol (lib_id "power:GND") (at 37.592 51.562 270) (unit 1)
@@
       (effects (font (size 1.27 1.27)) hide)
     )
+    (pin "1")
   )
   (symbol (lib_id "power:GND") (at 60.96 58.42 0) (unit 1)
@@
       (effects (font (size 1.27 1.27)) hide)
     )
+    (pin "1")
   )
   (symbol (lib_id "power:GND") (at 80.772 145.542 0) (unit 1)
@@
       (effects (font (size 1.27 1.27)) hide)
     )
+    (pin "1")
   )
   (symbol (lib_id "power:GND") (at 94.742 99.06 270) (unit 1)
@@
       (effects (font (size 1.27 1.27)) hide)
     )
+    (pin "1")
   )
   (symbol (lib_id "power:GND") (at 106.68 50.8 0) (unit 1)
@@
       (effects (font (size 1.27 1.27)) hide)
     )
+    (pin "1")
   )
   (symbol (lib_id "power:GND") (at 112.522 166.37 0) (unit 1)
@@
       (effects (font (size 1.27 1.27)) hide)
     )
+    (pin "1")
   )
   (symbol (lib_id "power:GND") (at 124.46 99.06 90) (unit 1)
@@
       (effects (font (size 1.27 1.27)) hide)
     )
+    (pin "1")
   )
   (symbol (lib_id "power:GND") (at 129.54 50.8 0) (unit 1)
@@
       (effects (font (size 1.27 1.27)) hide)
     )
+    (pin "1")
   )
   (symbol (lib_id "power:GND") (at 140.97 149.352 90) (unit 1)
@@
       (effects (font (size 1.27 1.27)) hide)
     )
+    (pin "1")
   )
   (symbol (lib_id "power:GND") (at 148.59 50.8 0) (unit 1)
@@
       (effects (font (size 1.27 1.27)) hide)
     )
+    (pin "1")
   )
   (symbol (lib_id "power:GND") (at 149.352 136.652 90) (unit 1)
@@
       (effects (font (size 1.27 1.27)) hide)
     )
+    (pin "1")
   )
   (symbol (lib_id "power:GND") (at 203.2 54.102 0) (unit 1)
@@
       (effects (font (size 1.27 1.27)) hide)
     )
+    (pin "1")
   )
   (symbol (lib_id "Device:R_Small") (at 142.24 134.112 270) (unit 1)
@@
       (effects (font (size 1.27 1.27)) hide)
     )
+    (pin "1")
+    (pin "2")
   )
   (symbol (lib_id "Device:R_Small") (at 143.51 139.192 270) (unit 1)
@@
       (effects (font (size 1.27 1.27)) hide)
     )
+    (pin "1")
+    (pin "2")
   )
   (symbol (lib_id "Device:C_Small") (at 68.58 113.792 90) (unit 1)
@@
       (effects (font (size 1.27 1.27)) hide)
     )
+    (pin "1")
+    (pin "2")
   )
   (symbol (lib_id "Device:C_Small") (at 69.342 126.492 90) (unit 1)
@@
       (effects (font (size 1.27 1.27)) hide)
     )
+    (pin "1")
+    (pin "2")
   )
   (symbol (lib_id "Device:C_Small") (at 74.422 116.332 90) (unit 1)
@@
       (effects (font (size 1.27 1.27)) hide)
     )
+    (pin "1")
+    (pin "2")
   )
   (symbol (lib_id "Device:C_Small") (at 74.422 129.032 90) (unit 1)
@@
       (effects (font (size 1.27 1.27)) hide)
     )
+    (pin "1")
+    (pin "2")
   )
   (symbol (lib_id "Device:C_Small") (at 100.33 99.06 270) (unit 1)
@@
       (effects (font (size 1.27 1.27)) hide)
     )
+    (pin "1")
+    (pin "2")
   )
   (symbol (lib_id "Device:C_Small") (at 103.632 43.18 180) (unit 1)
@@
       (effects (font (size 1.27 1.27)) hide)
     )
+    (pin "1")
+    (pin "2")
   )
   (symbol (lib_id "Device:C_Small") (at 109.982 43.18 180) (unit 1)
@@
       (effects (font (size 1.27 1.27)) hide)
     )
+    (pin "1")
+    (pin "2")
   )
   (symbol (lib_id "Device:C_Small") (at 118.872 99.06 270) (unit 1)
@@
       (effects (font (size 1.27 1.27)) hide)
     )
+    (pin "1")
+    (pin "2")
   )
   (symbol (lib_id "Device:C_Small") (at 145.542 43.18 180) (unit 1)
@@
       (effects (font (size 1.27 1.27)) hide)
     )
+    (pin "1")
+    (pin "2")
   )
   (symbol (lib_id "Device:C_Small") (at 150.622 108.712 90) (unit 1)
@@
       (effects (font (size 1.27 1.27)) hide)
     )
+    (pin "1")
+    (pin "2")
   )
   (symbol (lib_id "Device:C_Small") (at 150.622 118.872 90) (unit 1)
@@
       (effects (font (size 1.27 1.27)) hide)
     )
+    (pin "1")
+    (pin "2")
   )
   (symbol (lib_id "Device:C_Small") (at 152.4 43.18 180) (unit 1)
@@
       (effects (font (size 1.27 1.27)) hide)
     )
+    (pin "1")
+    (pin "2")
   )
   (symbol (lib_id "Device:C_Small") (at 155.702 111.252 90) (unit 1)
@@
       (effects (font (size 1.27 1.27)) hide)
     )
+    (pin "1")
+    (pin "2")
   )
   (symbol (lib_id "Device:C_Small") (at 155.702 116.332 90) (unit 1)
@@
       (effects (font (size 1.27 1.27)) hide)
     )
+    (pin "1")
+    (pin "2")
   )
   (symbol (lib_id "Device:FerriteBead_Small") (at 59.182 83.312 90) (unit 1)
@@
       (effects (font (size 1.27 1.27)) hide)
     )
+    (pin "1")
+    (pin "2")
   )
   (symbol (lib_id "Device:R_Pack04_Split") (at 203.2 36.322 0) (unit 1)
@@
       (effects (font (size 1.27 1.27)) hide)
     )
+    (pin "1")
+    (pin "8")
   )
   (symbol (lib_id "Device:LED") (at 203.2 46.482 90) (unit 1)
@@
       (effects (font (size 1.27 1.27)) hide)
     )
+    (pin "1")
+    (pin "2")
   )
   (symbol (lib_id "custom:MIC5363-3.3YMT") (at 129.54 41.402 0) (unit 1)
@@
       (effects (font (size 1.27 1.27)) hide)
     )
+    (pin "4")
+    (pin "3")
+    (pin "6")
+    (pin "1")
+    (pin "5")
+    (pin "2")
+    (pin "7")
   )
   (symbol (lib_id "custom:MG2040") (at 50.292 33.782 270) (unit 1)
@@
       (effects (font (size 1.27 1.27)) hide)
     )
+    (pin "1")
+    (pin "10")
+    (pin "11")
+    (pin "12")
+    (pin "13")
+    (pin "14")
+    (pin "15")
+    (pin "16")
+    (pin "17")
+    (pin "18")
+    (pin "19")
+    (pin "2")
+    (pin "20")
+    (pin "21")
+    (pin "3")
+    (pin "4")
+    (pin "5")
+    (pin "6")
+    (pin "7")
+    (pin "8")
+    (pin "9")
   )
   (symbol (lib_id "Connector:USB_C_Receptacle") (at 33.782 108.712 0) (unit 1)
@@
       (effects (font (size 1.27 1.27)) hide)
     )
+    (pin "A1")
+    (pin "A10")
+    (pin "A11")
+    (pin "A12")
+    (pin "A2")
+    (pin "A3")
+    (pin "A4")
+    (pin "A5")
+    (pin "A6")
+    (pin "A7")
+    (pin "A8")
+    (pin "A9")
+    (pin "B1")
+    (pin "B10")
+    (pin "B11")
+    (pin "B12")
+    (pin "B2")
+    (pin "B3")
+    (pin "B4")
+    (pin "B5")
+    (pin "B6")
+    (pin "B7")
+    (pin "B8")
+    (pin "B9")
+    (pin "S1")
   )
   (symbol (lib_id "custom:HD3SS3220") (at 109.982 131.572 0) (unit 1)
@@
       (effects (font (size 1.27 1.27)) hide)
     )
+    (pin "1")
+    (pin "2")
+    (pin "3")
+    (pin "4")
+    (pin "5")
+    (pin "6")
+    (pin "7")
+    (pin "8")
+    (pin "9")
+    (pin "10")
+    (pin "11")
+    (pin "12")
+    (pin "13")
+    (pin "14")
+    (pin "15")
+    (pin "16")
+    (pin "17")
+    (pin "18")
+    (pin "19")
+    (pin "20")
+    (pin "21")
+    (pin "22")
+    (pin "23")
+    (pin "24")
+    (pin "25")
+    (pin "26")
+    (pin "27")
+    (pin "28")
+    (pin "29")
+    (pin "30")
+    (pin "31")
   )
 )
